File: hardware/3w-rgb-led-connector-mk-3.0.sch (EAGLE design)
At the start: 13 parts

Commit message: teehee dongle
Parts:
- I2C: value M04JST-PTH -> M04JST_XH_RA; device A_butts:M04JST-PTH -> A_butts:M04JST_XH_RA
Changed lines of the file:
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@@
 <part name="B" library="A_butts" deviceset="M02" device="3.5MM-NO_SILK"/>
 <part name="U1" library="A_butts" deviceset="ARDUINO_SHIELD_SMALLER" device=""/>
-<part name="I2C" library="A_butts" deviceset="M04" device="JST-PTH"/>
+<part name="I2C" library="A_butts" deviceset="M04" device="JST_XH_RA" value="M04JST_XH_RA"/>
 <part name="GND1" library="A_butts" deviceset="GND" device=""/>
 <part name="GND2" library="A_butts" deviceset="GND" device=""/>
