File: hardware/3w-rgb-led-connector-mk-4.0.brd (EAGLE design)
At the start: 52 x 38 mm, 13 parts

Commit message: teehee dongle
Parts:
- removed B, G, R: M023.5MM-NO_SILK, A_butts:SCREWTERMINAL-3.5MM-2-NS
- removed C3: 10uF, A_butts:E2-5
- JP1: value (none) -> M06JST-XH-RA-PTH-LONG; device A_butts:1X08 -> A_butts:1X06-2.5MM-JST-XH-RA-LONG
- RGB+, RGB-: value M03JST-XH-RA-PTH -> M03JST-3-XH-RA-PTH-LONG; device A_butts:JST-3-XH-RA-PTH -> A_butts:JST-3-XH-RA-PTH-LONG
- moved JP1 33.1 mm to (7.00, 28.0), turned to 0 degrees
- moved RGB- 1.00 mm to (31.5, 28.0), flipped to the top
- moved RGB+ 0.50 mm to (42.0, 28.0), flipped to the top
Connections:
- net 5V: no longer C3.+, JP1.8
- net B+: now also JP1.6, RGB+.3; no longer B.2, RGB+.1
- net B-: now also JP1.5, RGB-.3; no longer B.1, RGB-.1
- net BLE_RST: no longer JP1.6
- net G+: now also JP1.4, RGB+.1; no longer G.2, RGB+.3
- net G-: now also JP1.3, RGB-.1; no longer G.1, RGB-.3
- net GND: no longer C3.-, JP1.7
- net MISO: no longer JP1.2
- net MOSI: no longer JP1.3
- net R+: now also JP1.2; no longer R.2
- net R-: now also JP1.1; no longer R.1
- net RDY: no longer JP1.5
- net REQ: no longer JP1.4
- net SCK: no longer JP1.1
Routing:
- net 5V: track 68.1 -> 53.7 mm
- net BLE_RST: track 23.1 -> 12.3 mm
- net MOSI: track 32.7 -> 22.9 mm
- net SCK: track 39.8 -> 30.1 mm
- net REQ: track 29.4 -> 19.7 mm
- net RDY: track 38.0 -> 28.3 mm
- net MISO: track 36.2 -> 26.5 mm
- net B+: track 25.4 -> 30.4 mm, vias 0 -> 1
- net G+: track 27.1 -> 32.1 mm
- net B-: track 19.0 -> 21.8 mm
- net R+: track 39.6 -> 41.8 mm
- net R-: track 32.8 -> 31.4 mm
- net G-: track 20.6 -> 21.9 mm
Other:
- outline, holes or cut-outs redrawn
