File: hardware/3w-rgb-led-connector-mk-7.0.sch (EAGLE design)
At the start: 8 parts, among them U1 SHEELD, U2 ADAFRUIT_9DOF_BREAKOUTHOLEY, U3 ADAFRUIT_BLE_UARTHOLEY-MOLEY

Commit message: dotstarstick
Parts:
- removed I2C_1: M04-I2CPTH-0.1IN, A_butts:M04-I2CPTH-0.1IN
- removed RXI, TXO: (no value), A_butts:JUMPER-PAD-3-NOFULL_BOX_SILK
- removed UART1: M06-UARTPTH-0.1IN, A_butts:M06-UARTPTH-0.1IN
- FRAME1: value (none) -> FRAME-LETTERNO_PACKAGE; VERSION v6.0 -> v7.0
- U2: value ADAFRUIT_9DOF_BREAKOUTHOLEY -> ADAFRUIT_BLUEFRUIT_LE_MICRO; device A_butts:ADAFRUIT_9DOF_BREAKOUTHOLEY -> A_butts:ADAFRUIT_BLUEFRUIT_LE_MICRO
- U3: value ADAFRUIT_BLE_UARTHOLEY-MOLEY -> ADAFRUIT_9DOF_BREAKOUT; device A_butts:ADAFRUIT_BLE_UARTHOLEY-MOLEY -> A_butts:ADAFRUIT_9DOF_BREAKOUT
Connections:
- removed net RX: TXO.1, U1.RX
- removed net RXI: RXI.2, U3.RXI, UART1.RXI
- removed net TX: RXI.1, U1.TX
- removed net TXO: TXO.2, U3.TXO, UART1.TXO
- new net 3.3V: U1.3.3V, U2.3V
- net 5V: now also U2.BAT; no longer I2C_1.VCC, U2.VIN, UART1.VIN
- net D2: no longer U3.CTS, UART1.CTS
- net D4: no longer U3.DFU
- net D5: now also U1.D5; no longer U1.*D5, U3.RTS, UART1.RTS
- net D6: now also U1.D6; no longer RXI.3, U1.*D6
- net D7: no longer TXO.3
- net D8: no longer U3.MOD
- net GND: no longer I2C_1.GND, UART1.GND
- net SCL: now also U2.3/SCL, U3.SCL; no longer I2C_1.SDA, U2.SCL
- net SDA: now also U2.2/SDA, U3.SDA; no longer I2C_1.SCL, U2.SDA
